Commit message: Merge seperated packages

File: urdf/rrbot.xacro (robot description, xacro)
@@ -12,7 +12,7 @@
   <xacro:property name="axel_offset" value="0.05" /> <!-- Space btw top of beam and the each joint -->
   <!-- Import all Gazebo-customization elements, including Gazebo colors -->
-  <xacro:include filename="$(find rrbot_description)/urdf/rrbot.gazebo" />
+  <xacro:include filename="$(find rifo_gazebo)/urdf/rrbot.gazebo" />
   <!-- Import Rviz colors -->
-  <xacro:include filename="$(find rrbot_description)/urdf/materials.xacro" />
+  <xacro:include filename="$(find rifo_gazebo)/urdf/materials.xacro" />
   <!-- Used for fixing robot to Gazebo 'base_link' -->
   <link name="world"/>
@@ -82,5 +82,5 @@
     <child link="link2"/>
     <origin xyz="0 0 ${height1}" rpy="0 0 0"/>
-    <axis xyz="0 -1 0"/>
+    <axis xyz="0 1 0"/>
     <dynamics damping="0.7"/>
   </joint>
@@ -113,5 +113,5 @@
     <child link="link3"/>
     <origin xyz="0 0 ${height2}" rpy="0 0 0"/>
-    <axis xyz="0 -1 0"/>
+    <axis xyz="0 1 0"/>
     <dynamics damping="0.7"/>
   </joint>

Commit message: Revise_Geometry

File: urdf/rrbot.xacro (robot description, xacro)
@@ -5,9 +5,9 @@
   <xacro:property name="PI" value="3.1415926535897931"/>
   <xacro:property name="mass" value="1" /> <!-- arbitrary value for mass -->
-  <xacro:property name="width" value="0.1" /> <!-- Square dimensions (widthxwidth) of beams -->
-  <xacro:property name="height1" value="0.25" /> <!-- Link 1 -->
-  <xacro:property name="height2" value="1" /> <!-- Link 2 -->
-  <xacro:property name="height3" value="1" /> <!-- Link 3 -->
-  <xacro:property name="camera_link" value="0.05" /> <!-- Size of square 'camera' box -->
+  <xacro:property name="r" value="0.05" /> <!-- Circle dimensions (PI*radius^2) of Rods -->
+  <xacro:property name="l1" value="0.25" /> <!-- Link 1 -->
+  <xacro:property name="l2" value="1" /> <!-- Link 2 -->
+  <xacro:property name="l3" value="1" /> <!-- Link 3 -->
+  <xacro:property name="camera_link" value="0.05" /> <!-- Size of square 'camera' cylinder -->
   <xacro:property name="axel_offset" value="0.05" /> <!-- Space btw top of beam and the each joint -->
   <!-- Import all Gazebo-customization elements, including Gazebo colors -->
@@ -27,23 +27,23 @@
   <link name="base">
     <collision>
-      <origin xyz="0 0 ${height1/2}" rpy="0 0 0"/>
-      <geometry>
-	      <box size="${width} ${width} ${height1}"/>
-      </geometry>
-    </collision>
-    <visual>
-      <origin xyz="0 0 ${height1/2}" rpy="0 0 0"/>
-      <geometry>
-        <box size="${width} ${width} ${height1}"/>
-      </geometry>
-      <material name="orange"/>
-    </visual>
-    <inertial>
-      <origin xyz="0 0 ${height1/2}" rpy="0 0 0"/>
-      <mass value="${mass}"/>
-      <inertia
-        ixx="${mass / 12.0 * (width*width + height1*height1)}" ixy="0.0" ixz="0.0"
-        iyy="${mass / 12.0 * (height1*height1 + width*width)}" iyz="0.0"
-        izz="${mass / 12.0 * (width*width + width*width)}"/>
+      <origin xyz="0 0 ${l1/2}" rpy="0 0 0"/>
+      <geometry>
+	      <cylinder length="${l1}" radius="${r}"/>
+      </geometry>
+    </collision>
+    <visual>
+      <origin xyz="0 0 ${l1/2}" rpy="0 0 0"/>
+      <geometry>
+        <cylinder length="${l1}" radius="${r}"/>
+      </geometry>
+      <material name="orange"/>
+    </visual>
+    <inertial>
+      <origin xyz="0 0 ${l1/2}" rpy="0 0 0"/>
+      <mass value="${mass}"/>
+      <inertia
+	  ixx="${mass / 12.0 * (3*r*r + l1*l1)}" ixy="0.0" ixz="0.0"
+	  iyy="${mass / 12.0 * (l1*l1 + 3*r*r)}" iyz="0.0"
+	  izz="${mass / 12.0 * (3*r*r)}"/>
     </inertial>
   </link>
@@ -51,5 +51,5 @@
     <parent link="base"/>
     <child link="link1"/>
-    <origin xyz="0 0 ${height1}" rpy="0 0 0"/>
+    <origin xyz="0 0 ${l1}" rpy="0 0 0"/>
     <axis xyz="0 0 1"/>
     <dynamics damping="0.7"/>
@@ -57,23 +57,23 @@
   <link name="link1">
     <collision>
-      <origin xyz="0 0 ${height1/2}" rpy="0 0 0"/>
-      <geometry>
-	      <box size="${width} ${width} ${height1}"/>
-      </geometry>
-    </collision>
-    <visual>
-      <origin xyz="0 0 ${height1/2}" rpy="0 0 0"/>
-      <geometry>
-	      <box size="${width} ${width} ${height1}"/>
-      </geometry>
-      <material name="orange"/>
-    </visual>
-    <inertial>
-      <origin xyz="0 0 ${height1/2}" rpy="0 0 0"/>
-      <mass value="${mass}"/>
-      <inertia
-	  ixx="${mass / 12.0 * (width*width + height1*height1)}" ixy="0.0" ixz="0.0"
-	  iyy="${mass / 12.0 * (height1*height1 + width*width)}" iyz="0.0"
-	  izz="${mass / 12.0 * (width*width + width*width)}"/>
+      <origin xyz="0 0 ${l1/2}" rpy="0 0 0"/>
+      <geometry>
+	      <cylinder length="${l1}" radius="${r}"/>
+      </geometry>
+    </collision>
+    <visual>
+      <origin xyz="0 0 ${l1/2}" rpy="0 0 0"/>
+      <geometry>
+	      <cylinder length="${l1}" radius="${r}"/>
+      </geometry>
+      <material name="orange"/>
+    </visual>
+    <inertial>
+      <origin xyz="0 0 ${l1/2}" rpy="0 0 0"/>
+      <mass value="${mass}"/>
+      <inertia
+	  ixx="${mass / 12.0 * (3*r*r + l1*l1)}" ixy="0.0" ixz="0.0"
+	  iyy="${mass / 12.0 * (l1*l1 + 3*r*r)}" iyz="0.0"
+	  izz="${mass / 12.0 * (3*r*r)}"/>
     </inertial>
   </link>
@@ -81,5 +81,5 @@
     <parent link="link1"/>
     <child link="link2"/>
-    <origin xyz="0 0 ${height1}" rpy="0 0 0"/>
+    <origin xyz="0 0 ${l1}" rpy="0 0 0"/>
     <axis xyz="0 1 0"/>
     <dynamics damping="0.7"/>
@@ -88,23 +88,23 @@
   <link name="link2">
     <collision>
-      <origin xyz="0 0 ${height2/2}" rpy="0 0 0"/>
-      <geometry>
-	<box size="${width} ${width} ${height2}"/>
-      </geometry>
-    </collision>
-    <visual>
-      <origin xyz="0 0 ${height2/2}" rpy="0 0 0"/>
-      <geometry>
-	<box size="${width} ${width} ${height2}"/>
+      <origin xyz="0 0 ${l2/2}" rpy="0 0 0"/>
+      <geometry>
+	<cylinder length="${l2}" radius="${r}"/>
+      </geometry>
+    </collision>
+    <visual>
+      <origin xyz="0 0 ${l2/2}" rpy="0 0 0"/>
+      <geometry>
+	<cylinder length="${l2}" radius="${r}"/>
       </geometry>
       <material name="black"/>
     </visual>
     <inertial>
-      <origin xyz="0 0 ${height2/2}" rpy="0 0 0"/>
-      <mass value="${mass}"/>
-      <inertia
-	  ixx="${mass / 12.0 * (width*width + height2*height2)}" ixy="0.0" ixz="0.0"
-	  iyy="${mass / 12.0 * (height2*height2 + width*width)}" iyz="0.0"
-	  izz="${mass / 12.0 * (width*width + width*width)}"/>
+      <origin xyz="0 0 ${l2/2}" rpy="0 0 0"/>
+      <mass value="${mass}"/>
+      <inertia
+	  ixx="${mass / 12.0 * (3*r*r + l2*l2)}" ixy="0.0" ixz="0.0"
+	  iyy="${mass / 12.0 * (l2*l2 + 3*r*r)}" iyz="0.0"
+	  izz="${mass / 12.0 * (3*r*r)}"/>
     </inertial>
   </link>
@@ -112,5 +112,5 @@
     <parent link="link2"/>
     <child link="link3"/>
-    <origin xyz="0 0 ${height2}" rpy="0 0 0"/>
+    <origin xyz="0 0 ${l2}" rpy="0 0 0"/>
     <axis xyz="0 1 0"/>
     <dynamics damping="0.7"/>
@@ -119,23 +119,23 @@
   <link name="link3">
     <collision>
-      <origin xyz="0 0 ${height3/2}" rpy="0 0 0"/>
-      <geometry>
-	<box size="${width} ${width} ${height3}"/>
-      </geometry>
-    </collision>
-    <visual>
-      <origin xyz="0 0 ${height3/2}" rpy="0 0 0"/>
-      <geometry>
-	<box size="${width} ${width} ${height3}"/>
-      </geometry>
-      <material name="orange"/>
-    </visual>
-    <inertial>
-      <origin xyz="0 0 ${height3/2}" rpy="0 0 0"/>
-      <mass value="${mass}"/>
-      <inertia
-	  ixx="${mass / 12.0 * (width*width + height3*height3)}" ixy="0.0" ixz="0.0"
-	  iyy="${mass / 12.0 * (height3*height3 + width*width)}" iyz="0.0"
-	  izz="${mass / 12.0 * (width*width + width*width)}"/>
+      <origin xyz="0 0 ${l3/2}" rpy="0 0 0"/>
+      <geometry>
+	<cylinder length="${l3}" radius="${r}"/>
+      </geometry>
+    </collision>
+    <visual>
+      <origin xyz="0 0 ${l3/2}" rpy="0 0 0"/>
+      <geometry>
+	<cylinder length="${l3}" radius="${r}"/>
+      </geometry>
+      <material name="orange"/>
+    </visual>
+    <inertial>
+      <origin xyz="0 0 ${l3/2}" rpy="0 0 0"/>
+      <mass value="${mass}"/>
+      <inertia
+	  ixx="${mass / 12.0 * (3*r*r + l3*l3)}" ixy="0.0" ixz="0.0"
+	  iyy="${mass / 12.0 * (l3*l3 + 3*r*r)}" iyz="0.0"
+	  izz="${mass / 12.0 * (3*r*r)}"/>
     </inertial>
   </link>
@@ -143,17 +143,18 @@
     <parent link="link3"/>
     <child link="end_effector"/>
-    <origin xyz="0 0 ${height2}" rpy="0 0 0"/>
-  </joint>
+    <origin xyz="0 0 ${l2}" rpy="0 0 0"/>
+  </joint>
+<!-- End_effector -->
   <link name="end_effector">
     <collision>
-      <origin xyz="0 0 0" rpy="0 0 0"/>
-      <geometry>
-	      <box size="0 0 0"/>
-      </geometry>
-    </collision>
-    <visual>
-      <origin xyz="0 0 0" rpy="0 0 0"/>
-      <geometry>
-	      <box size="0 0 0"/>
+      <origin xyz="0 0.5 0.125" rpy="0 0 0"/>
+      <geometry>
+	      <box size="0.25 0.25 0.25"/>
+      </geometry>
+    </collision>
+    <visual>
+      <origin xyz="0 0.5 0.125" rpy="0 0 0"/>
+      <geometry>
+	      <box size="0.25 0.25 0.25"/>
       </geometry>
       <material name="orange"/>
@@ -163,7 +164,7 @@
       <mass value="0"/>
       <inertia
-	  ixx="0" ixy="0.0" ixz="0.0"
-	  iyy="0" iyz="0.0"
-	  izz="0"/>
+	  ixx="0.01" ixy="0.0" ixz="0.0"
+	  iyy="0.01" iyz="0.0"
+	  izz="0.01"/>
     </inertial>
   </link>

Commit message: Add_Gripper

File: urdf/rrbot.xacro (robot description, xacro)
@@ -56,4 +56,27 @@
   </joint>
   <link name="link1">
+<!-- Sphere -->
+    <collision>
+      <origin xyz="0 0 0" rpy="0 0 0"/>
+      <geometry>
+	  <sphere radius="0.06"/>
+      </geometry>
+    </collision>
+    <visual>
+      <origin xyz="0 0 0" rpy="0 0 0"/>
+      <geometry>
+	 <sphere radius="0.06"/>
+      </geometry>
+      <material name="Black"/>
+    </visual>
+    <inertial>
+      <origin xyz="0 0 0" rpy="0 0 0"/>
+      <mass value="${mass}"/>
+      <inertia
+	  ixx="0.001" ixy="0.0" ixz="0.0"
+	  iyy="0.001" iyz="0.0"
+	  izz="0.001"/>
+    </inertial>
+<!-- Cylinder -->
     <collision>
       <origin xyz="0 0 ${l1/2}" rpy="0 0 0"/>
@@ -86,5 +109,28 @@
   </joint>
   <!-- Middle Link -->
-  <link name="link2">
+<link name="link2">
+<!-- Sphere -->
+    <collision>
+      <origin xyz="0 0 0" rpy="0 0 0"/>
+      <geometry>
+	  <sphere radius="0.06"/>
+      </geometry>
+    </collision>
+    <visual>
+      <origin xyz="0 0 0" rpy="0 0 0"/>
+      <geometry>
+	 <sphere radius="0.06"/>
+      </geometry>
+      <material name="orange"/>
+    </visual>
+    <inertial>
+      <origin xyz="0 0 0" rpy="0 0 0"/>
+      <mass value="${mass}"/>
+      <inertia
+	  ixx="0.001" ixy="0.0" ixz="0.0"
+	  iyy="0.001" iyz="0.0"
+	  izz="0.001"/>
+    </inertial>
+<!-- Cylinder -->
     <collision>
       <origin xyz="0 0 ${l2/2}" rpy="0 0 0"/>
@@ -118,4 +164,27 @@
   <!-- Top Link -->
   <link name="link3">
+<!-- Sphere -->
+    <collision>
+      <origin xyz="0 0 0" rpy="0 0 0"/>
+      <geometry>
+	  <sphere radius="0.06"/>
+      </geometry>
+    </collision>
+    <visual>
+      <origin xyz="0 0 0" rpy="0 0 0"/>
+      <geometry>
+	 <sphere radius="0.06"/>
+      </geometry>
+      <material name="orange"/>
+    </visual>
+    <inertial>
+      <origin xyz="0 0 0" rpy="0 0 0"/>
+      <mass value="${mass}"/>
+      <inertia
+	  ixx="0.001" ixy="0.0" ixz="0.0"
+	  iyy="0.001" iyz="0.0"
+	  izz="0.001"/>
+    </inertial>
+<!-- Cylinder -->
     <collision>
       <origin xyz="0 0 ${l3/2}" rpy="0 0 0"/>
@@ -147,24 +216,66 @@
 <!-- End_effector -->
   <link name="end_effector">
-    <collision>
-      <origin xyz="0 0.5 0.125" rpy="0 0 0"/>
-      <geometry>
-	      <box size="0.25 0.25 0.25"/>
-      </geometry>
-    </collision>
-    <visual>
-      <origin xyz="0 0.5 0.125" rpy="0 0 0"/>
-      <geometry>
-	      <box size="0.25 0.25 0.25"/>
-      </geometry>
-      <material name="orange"/>
-    </visual>
-    <inertial>
-      <origin xyz="0 0 0" rpy="0 0 0"/>
+   <collision>
+      <origin xyz="0 0 0.03125" rpy="0 0 0"/>
+      <geometry>
+	      <box size="0.1 0.1 0.0625"/>
+      </geometry>
+    </collision>
+    <visual>
+      <origin xyz="0 0 0.03125" rpy="0 0 0"/>
+      <geometry>
+	      <box size="0.1 0.1 0.0625"/>
+      </geometry>
+      <material name="orange"/>
+    </visual>
+    <inertial>
+      <origin xyz="0 0 0.03125" rpy="0 0 0"/>
       <mass value="0"/>
       <inertia
-	  ixx="0.01" ixy="0.0" ixz="0.0"
-	  iyy="0.01" iyz="0.0"
-	  izz="0.01"/>
+	  ixx="0.00052" ixy="0.0" ixz="0.0"
+	  iyy="0.00052" iyz="0.0"
+	  izz="0.0008"/>
+    </inertial>
+    <collision>
+      <origin xyz="0 0.07 0.125" rpy="0 0 0"/>
+      <geometry>
+	      <box size="0.05 0.05 0.25"/>
+      </geometry>
+    </collision>
+    <visual>
+      <origin xyz="0 0.07 0.125" rpy="0 0 0"/>
+      <geometry>
+	      <box size="0.05 0.05 0.25"/>
+      </geometry>
+      <material name="orange"/>
+    </visual>
+    <inertial>
+      <origin xyz="0 0.07 0.125" rpy="0 0 0"/>
+      <mass value="0"/>
+      <inertia
+	  ixx="0.0002" ixy="0.0" ixz="0.0"
+	  iyy="0.0002" iyz="0.0"
+	  izz="0.0004"/>
+    </inertial>
+<collision>
+      <origin xyz="0 -0.07 0.125" rpy="0 0 0"/>
+      <geometry>
+	      <box size="0.05 0.05 0.25"/>
+      </geometry>
+    </collision>
+    <visual>
+      <origin xyz="0 -0.07 0.125" rpy="0 0 0"/>
+      <geometry>
+	      <box size="0.05 0.05 0.25"/>
+      </geometry>
+      <material name="orange"/>
+    </visual>
+    <inertial>
+      <origin xyz="0 -0.07 0.125" rpy="0 0 0"/>
+      <mass value="0"/>
+      <inertia
+	  ixx="0.0002" ixy="0.0" ixz="0.0"
+	  iyy="0.0002" iyz="0.0"
+	  izz="0.0004"/>
     </inertial>
   </link>
